File: PCB Design.kicad_pcb (KiCad board)
At the start: 2 copper layers, 24 parts, among them SW1 SW_Push, U1 ATmega32U4-AU, Y1 16MHz

Commit message: Preliminary PCB layout for 4 switch board
Parts:
- C3, C4, C5, C6, C7, F1, R1, R2, R3, R4, SW1, USB1: moved to B.Cu
- moved R2 129.7 mm to (27.1, 44.1), turned to 270 degrees
- moved USB1 121.8 mm to (25.9, 34.4), turned to 270 degrees
- moved C4 120.0 mm to (35.4, 66.9)
- moved C7 119.6 mm to (27.2, 48.6), turned to 90 degrees
- moved R3 114.7 mm to (30.5, 48.6), turned to 90 degrees
- moved SW1 112.8 mm to (23.6, 66.4), turned to 180 degrees
- moved F1 111.1 mm to (20.6, 49.1), turned to 270 degrees
- moved R1 107.7 mm to (24.1, 44.1), turned to 90 degrees
- moved C6 105.4 mm to (35.2, 44.6), turned to 90 degrees
- moved C3 95.7 mm to (42.8, 66.9), turned to 180 degrees
- moved R4 95.6 mm to (47.1, 62.9), turned to 270 degrees
- moved C5 94.1 mm to (42.7, 44.6), turned to 270 degrees
- moved C2 28.6 mm to (47.9, 53.8), turned to 90 degrees
- moved C1 25.7 mm to (29.2, 58.8)
- moved U1 13.2 mm to (39.1, 56.9)
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Other:
- board outline added: 71.1 x 38.2 mm

Commit message: Editing schematic to include all 48 keys
Other:
- net class Default: trace_width 0.25 -> 0.254
- net class Power added: clearance 0.2, trace_width 0.381, via_dia 0.8, via_drill 0.4
Changed lines of the file:
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@@
   )
   (setup
-    (last_trace_width 0.25)
+    (last_trace_width 0.254)
     (trace_clearance 0.2)
     (zone_clearance 0.508)
@@
   (net_class Default "This is the default net class."
     (clearance 0.2)
-    (trace_width 0.25)
+    (trace_width 0.254)
     (via_dia 0.8)
     (via_drill 0.4)
     (uvia_dia 0.3)
     (uvia_drill 0.1)
-    (add_net +5V)
     (add_net D+)
     (add_net D-)
-    (add_net GND)
     (add_net "Net-(C5-Pad2)")
     (add_net "Net-(C6-Pad2)")
@@
     (add_net "Net-(U1-Pad9)")
     (add_net "Net-(USB1-Pad2)")
-    (add_net VCC)
     (add_net col0)
     (add_net col1)
@@
     (add_net row1)
   )
+  (net_class Power ""
+    (clearance 0.2)
+    (trace_width 0.381)
+    (via_dia 0.8)
+    (via_drill 0.4)
+    (uvia_dia 0.3)
+    (uvia_drill 0.1)
+    (add_net +5V)
+    (add_net GND)
+    (add_net VCC)
+  )
   (module Crystal:Crystal_SMD_3225-4Pin_3.2x2.5mm (layer B.Cu)

Commit message: Diode layout completed
Parts:
- added D10: D_Small, Diode_SMD:D_SOD-123, B.Cu at (108.0, 60.3)
- added D11: D_Small, Diode_SMD:D_SOD-123, B.Cu at (108.0, 79.4)
- added D12: D_Small, Diode_SMD:D_SOD-123, B.Cu at (108.0, 98.4)
- added D13: D_Small, Diode_SMD:D_SOD-123, B.Cu at (127.0, 41.3)
- added D14: D_Small, Diode_SMD:D_SOD-123, B.Cu at (127.0, 60.3)
- added D15: D_Small, Diode_SMD:D_SOD-123, B.Cu at (127.0, 79.4)
- added D16: D_Small, Diode_SMD:D_SOD-123, B.Cu at (127.0, 98.4)
- added D17: D_Small, Diode_SMD:D_SOD-123, B.Cu at (146.1, 41.3)
- added D18: D_Small, Diode_SMD:D_SOD-123, B.Cu at (146.1, 60.3)
- added D19: D_Small, Diode_SMD:D_SOD-123, B.Cu at (146.1, 79.4)
- added D20: D_Small, Diode_SMD:D_SOD-123, B.Cu at (146.1, 98.4)
- added D21: D_Small, Diode_SMD:D_SOD-123, B.Cu at (165.1, 41.3)
- added D22: D_Small, Diode_SMD:D_SOD-123, B.Cu at (165.1, 60.3)
- added D23: D_Small, Diode_SMD:D_SOD-123, B.Cu at (165.1, 79.4)
- added D24: D_Small, Diode_SMD:D_SOD-123, B.Cu at (165.1, 98.4)
- added D25: D_Small, Diode_SMD:D_SOD-123, B.Cu at (184.2, 41.3)
- added D26: D_Small, Diode_SMD:D_SOD-123, B.Cu at (184.2, 60.3)
- added D27: D_Small, Diode_SMD:D_SOD-123, B.Cu at (184.2, 79.4)
- added D28: D_Small, Diode_SMD:D_SOD-123, B.Cu at (184.2, 98.4)
- added D29: D_Small, Diode_SMD:D_SOD-123, B.Cu at (203.2, 41.3)
- added D30: D_Small, Diode_SMD:D_SOD-123, B.Cu at (203.2, 60.3)
- added D31: D_Small, Diode_SMD:D_SOD-123, B.Cu at (203.2, 79.4)
- added D32: D_Small, Diode_SMD:D_SOD-123, B.Cu at (203.2, 98.4)
- added D33: D_Small, Diode_SMD:D_SOD-123, B.Cu at (222.2, 41.3)
- added D34: D_Small, Diode_SMD:D_SOD-123, B.Cu at (222.2, 60.3)
- added D35: D_Small, Diode_SMD:D_SOD-123, B.Cu at (222.2, 79.4)
- added D36: D_Small, Diode_SMD:D_SOD-123, B.Cu at (222.2, 98.4)
- added D37: D_Small, Diode_SMD:D_SOD-123, B.Cu at (241.3, 41.3)
- added D38: D_Small, Diode_SMD:D_SOD-123, B.Cu at (241.3, 60.3)
- added D39: D_Small, Diode_SMD:D_SOD-123, B.Cu at (241.3, 79.4)
- added D40: D_Small, Diode_SMD:D_SOD-123, B.Cu at (241.3, 98.4)
- added D41: D_Small, Diode_SMD:D_SOD-123, B.Cu at (260.4, 41.3)
- added D42: D_Small, Diode_SMD:D_SOD-123, B.Cu at (260.4, 60.3)
- added D43: D_Small, Diode_SMD:D_SOD-123, B.Cu at (260.4, 79.4)
- added D44: D_Small, Diode_SMD:D_SOD-123, B.Cu at (260.4, 98.4)
- added D45: D_Small, Diode_SMD:D_SOD-123, B.Cu at (279.4, 41.3)
- added D46: D_Small, Diode_SMD:D_SOD-123, B.Cu at (279.4, 60.3)
- added D47: D_Small, Diode_SMD:D_SOD-123, B.Cu at (279.4, 79.4)
- added D48: D_Small, Diode_SMD:D_SOD-123, B.Cu at (279.4, 98.4)
- added D5: D_Small, Diode_SMD:D_SOD-123, B.Cu at (69.8, 79.4)
- added D6: D_Small, Diode_SMD:D_SOD-123, B.Cu at (69.8, 98.4)
- added D7: D_Small, Diode_SMD:D_SOD-123, B.Cu at (88.9, 79.4)
- added D8: D_Small, Diode_SMD:D_SOD-123, B.Cu at (88.9, 98.4)
- added D9: D_Small, Diode_SMD:D_SOD-123, B.Cu at (108.0, 41.3)
- added MX10: MX-NoLED, MX_Alps_Hybrid1:MX-1U-NoLED, F.Cu at (100.0, 60.3)
- added MX11: MX-NoLED, MX_Alps_Hybrid1:MX-1U-NoLED, F.Cu at (100.0, 79.4)
- added MX12: MX-NoLED, MX_Alps_Hybrid1:MX-1U-NoLED, F.Cu at (100.0, 98.4)
- added MX13: MX-NoLED, MX_Alps_Hybrid1:MX-1U-NoLED, F.Cu at (119.1, 41.3)
- added MX14: MX-NoLED, MX_Alps_Hybrid1:MX-1U-NoLED, F.Cu at (119.1, 60.3)
- added MX15: MX-NoLED, MX_Alps_Hybrid1:MX-1U-NoLED, F.Cu at (119.1, 79.4)
- added MX16: MX-NoLED, MX_Alps_Hybrid1:MX-1U-NoLED, F.Cu at (119.1, 98.4)
- added MX17: MX-NoLED, MX_Alps_Hybrid1:MX-1U-NoLED, F.Cu at (138.1, 41.3)
- added MX18: MX-NoLED, MX_Alps_Hybrid1:MX-1U-NoLED, F.Cu at (138.1, 60.3)
- added MX19: MX-NoLED, MX_Alps_Hybrid1:MX-1U-NoLED, F.Cu at (138.1, 79.4)
- added MX20: MX-NoLED, MX_Alps_Hybrid1:MX-1U-NoLED, F.Cu at (138.1, 98.4)
- added MX21: MX-NoLED, MX_Alps_Hybrid1:MX-1U-NoLED, F.Cu at (157.2, 41.3)
- added MX22: MX-NoLED, MX_Alps_Hybrid1:MX-1U-NoLED, F.Cu at (157.2, 60.3)
- added MX23: MX-NoLED, MX_Alps_Hybrid1:MX-1U-NoLED, F.Cu at (157.2, 79.4)
- added MX24: MX-NoLED, MX_Alps_Hybrid1:MX-1U-NoLED, F.Cu at (157.2, 98.4)
- added MX25: MX-NoLED, MX_Alps_Hybrid1:MX-1U-NoLED, F.Cu at (176.2, 41.3)
- added MX26: MX-NoLED, MX_Alps_Hybrid1:MX-1U-NoLED, F.Cu at (176.2, 60.3)
- added MX27: MX-NoLED, MX_Alps_Hybrid1:MX-1U-NoLED, F.Cu at (176.2, 79.4)
- added MX28: MX-NoLED, MX_Alps_Hybrid1:MX-1U-NoLED, F.Cu at (176.2, 98.4)
- added MX29: MX-NoLED, MX_Alps_Hybrid1:MX-1U-NoLED, F.Cu at (195.3, 41.3)
- added MX30: MX-NoLED, MX_Alps_Hybrid1:MX-1U-NoLED, F.Cu at (195.3, 60.3)
- added MX31: MX-NoLED, MX_Alps_Hybrid1:MX-1U-NoLED, F.Cu at (195.3, 79.4)
- added MX32: MX-NoLED, MX_Alps_Hybrid1:MX-1U-NoLED, F.Cu at (195.3, 98.4)
- added MX33: MX-NoLED, MX_Alps_Hybrid1:MX-1U-NoLED, F.Cu at (214.3, 41.3)
- added MX34: MX-NoLED, MX_Alps_Hybrid1:MX-1U-NoLED, F.Cu at (214.3, 60.3)
- added MX35: MX-NoLED, MX_Alps_Hybrid1:MX-1U-NoLED, F.Cu at (214.3, 79.4)
- added MX36: MX-NoLED, MX_Alps_Hybrid1:MX-1U-NoLED, F.Cu at (214.3, 98.4)
- added MX37: MX-NoLED, MX_Alps_Hybrid1:MX-1U-NoLED, F.Cu at (233.4, 41.3)
- added MX38: MX-NoLED, MX_Alps_Hybrid1:MX-1U-NoLED, F.Cu at (233.4, 60.3)
- added MX39: MX-NoLED, MX_Alps_Hybrid1:MX-1U-NoLED, F.Cu at (233.4, 79.4)
- added MX40: MX-NoLED, MX_Alps_Hybrid1:MX-1U-NoLED, F.Cu at (233.4, 98.4)
- added MX41: MX-NoLED, MX_Alps_Hybrid1:MX-1U-NoLED, F.Cu at (252.4, 41.3)
- added MX42: MX-NoLED, MX_Alps_Hybrid1:MX-1U-NoLED, F.Cu at (252.4, 60.3)
- added MX43: MX-NoLED, MX_Alps_Hybrid1:MX-1U-NoLED, F.Cu at (252.4, 79.4)
- added MX44: MX-NoLED, MX_Alps_Hybrid1:MX-1U-NoLED, F.Cu at (252.4, 98.4)
- added MX45: MX-NoLED, MX_Alps_Hybrid1:MX-1U-NoLED, F.Cu at (271.5, 41.3)
- added MX46: MX-NoLED, MX_Alps_Hybrid1:MX-1U-NoLED, F.Cu at (271.5, 60.3)
- added MX47: MX-NoLED, MX_Alps_Hybrid1:MX-1U-NoLED, F.Cu at (271.5, 79.4)
- added MX48: MX-NoLED, MX_Alps_Hybrid1:MX-1U-NoLED, F.Cu at (271.5, 98.4)
- added MX5: MX-NoLED, MX_Alps_Hybrid1:MX-1U-NoLED, F.Cu at (61.9, 79.4)
- added MX6: MX-NoLED, MX_Alps_Hybrid1:MX-1U-NoLED, F.Cu at (61.9, 98.4)
- added MX7: MX-NoLED, MX_Alps_Hybrid1:MX-1U-NoLED, F.Cu at (81.0, 79.4)
- added MX8: MX-NoLED, MX_Alps_Hybrid1:MX-1U-NoLED, F.Cu at (81.0, 98.4)
- added MX9: MX-NoLED, MX_Alps_Hybrid1:MX-1U-NoLED, F.Cu at (100.0, 41.3)
- moved D3 28.8 mm to (88.9, 41.3)
- moved MX3 28.8 mm to (81.0, 41.3)
- moved D2 25.1 mm to (69.8, 60.3)
- moved MX2 25.1 mm to (61.9, 60.3)
- moved D4 1.92 mm to (88.9, 60.3)
- moved MX4 1.92 mm to (81.0, 60.3)
- moved MX1 1.92 mm to (61.9, 41.3)
- moved D1 1.92 mm to (69.8, 41.3)
Other:
- board outline removed

Commit message: Pre-trace, need to figure out how to place microcontroller on board itself
Parts:
- moved R4 1.08 mm to (47.6, 61.9)
- moved C3 1.05 mm to (42.8, 65.9)
- moved C4 1.05 mm to (35.4, 65.9)
- moved C1 0.95 mm to (30.2, 58.8)
- moved C2 0.25 mm to (47.6, 53.8)
Other:
- board outline added: 228.6 x 76.2 mm
Changed lines of the file:
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@@
   (general
     (thickness 1.6)
-    (drawings 0)
+    (drawings 8)
     (tracks 0)
     (zones 0)
@@
   )
   (module Resistor_SMD:R_0805_2012Metric (layer B.Cu)
-    (at 47.117 62.865 270)
+    (at 47.625 61.9125 270)
     (descr "Resistor SMD 0805 (2012 Metric), square (rectangular) end terminal, IPC_7351 nominal, (Body size source: https://docs.google.com/spreadsheets/d/1BsfQQcO9C6DZCsRaXUlFlo91Tg2WpOkGARC1WS5S8t0/edit?usp=sharing), generated with kicad-footprint-generator")
     (tags resistor)
@@
   )
   (module Capacitor_SMD:C_0805_2012Metric (layer B.Cu)
-    (at 35.433 66.929)
+    (at 35.433 65.88125)
     (descr "Capacitor SMD 0805 (2012 Metric), square (rectangular) end terminal, IPC_7351 nominal, (Body size source: https://docs.google.com/spreadsheets/d/1BsfQQcO9C6DZCsRaXUlFlo91Tg2WpOkGARC1WS5S8t0/edit?usp=sharing), generated with kicad-footprint-generator")
     (tags capacitor)
@@
   )
   (module Capacitor_SMD:C_0805_2012Metric (layer B.Cu)
-    (at 42.799 66.929 180)
+    (at 42.799 65.88125 180)
     (descr "Capacitor SMD 0805 (2012 Metric), square (rectangular) end terminal, IPC_7351 nominal, (Body size source: https://docs.google.com/spreadsheets/d/1BsfQQcO9C6DZCsRaXUlFlo91Tg2WpOkGARC1WS5S8t0/edit?usp=sharing), generated with kicad-footprint-generator")
     (tags capacitor)
@@
   )
   (module Capacitor_SMD:C_0805_2012Metric (layer B.Cu)
-    (at 47.879 53.848 90)
+    (at 47.625 53.848 90)
     (descr "Capacitor SMD 0805 (2012 Metric), square (rectangular) end terminal, IPC_7351 nominal, (Body size source: https://docs.google.com/spreadsheets/d/1BsfQQcO9C6DZCsRaXUlFlo91Tg2WpOkGARC1WS5S8t0/edit?usp=sharing), generated with kicad-footprint-generator")
     (tags capacitor)
@@
   )
   (module Capacitor_SMD:C_0805_2012Metric (layer B.Cu)
-    (at 29.21 58.7525 90)
+    (at 30.1625 58.7525 90)
     (descr "Capacitor SMD 0805 (2012 Metric), square (rectangular) end terminal, IPC_7351 nominal, (Body size source: https://docs.google.com/spreadsheets/d/1BsfQQcO9C6DZCsRaXUlFlo91Tg2WpOkGARC1WS5S8t0/edit?usp=sharing), generated with kicad-footprint-generator")
     (tags capacitor)
@@
     )
   )
+  (gr_line (start 54.76875 31.75) (end 278.60625 31.75) (layer Edge.Cuts) (width 0.05))
+  (gr_line (start 52.3875 105.56875) (end 52.3875 34.13125) (layer Edge.Cuts) (width 0.05))
+  (gr_line (start 278.60625 107.95) (end 54.76875 107.95) (layer Edge.Cuts) (width 0.05))
+  (gr_line (start 280.9875 34.13125) (end 280.9875 105.56875) (layer Edge.Cuts) (width 0.05))
+  (gr_arc (start 54.76875 105.56875) (end 52.3875 105.56875) (angle -90) (layer Edge.Cuts) (width 0.05))
+  (gr_arc (start 54.76875 34.13125) (end 54.76875 31.75) (angle -90) (layer Edge.Cuts) (width 0.05))
+  (gr_arc (start 278.60625 105.56875) (end 278.60625 107.95) (angle -90) (layer Edge.Cuts) (width 0.05))
+  (gr_arc (start 278.60625 34.13125) (end 280.9875 34.13125) (angle -90) (layer Edge.Cuts) (width 0.05))
 )

Commit message: Preliminary PCB completed
Parts:
- moved U1 113.4 mm to (144.3, 99.4)
- moved C2 113.3 mm to (152.8, 96.1)
- moved C1 113.2 mm to (136.1, 98.6)
- moved R4 113.1 mm to (152.8, 103.3)
- moved C4 112.6 mm to (140.1, 107.3)
- moved C3 111.9 mm to (146.5, 108.1)
- moved C5 111.5 mm to (147.7, 81.9)
- moved C6 111.5 mm to (140.2, 81.9)
- moved Y1 111.5 mm to (144.0, 81.9)
- moved C7 111.1 mm to (126.5, 98.4)
- moved R3 111.1 mm to (129.8, 98.4)
- moved SW1 59.2 mm to (48.8, 120.0)
- moved R1 44.4 mm to (47.4, 81.9)
- moved R2 44.4 mm to (50.3, 81.9)
- moved F1 40.3 mm to (44.1, 81.9)
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
Commit message: Done with switch traces
Routing:
- net row1: track 0.00 -> 250.5 mm
- net row3: track 0.00 -> 241.6 mm
- net row2: track 0.00 -> 230.7 mm
- net row0: track 0.00 -> 224.9 mm
- net col6: track 0.00 -> 69.0 mm
- net col5: track 0.00 -> 59.6 mm
- net col4: track 0.00 -> 58.1 mm
- net col10: track 0.00 -> 57.5 mm
- net col8: track 0.00 -> 57.3 mm
- net col7: track 0.00 -> 57.2 mm
- net col9: track 0.00 -> 57.2 mm
- net col3: track 0.00 -> 57.2 mm
- net col2: track 0.00 -> 57.2 mm
- net col11: track 0.00 -> 57.2 mm
- net col1: track 0.00 -> 57.2 mm
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
Commit message: Working on trace pt.1
Parts:
- moved D1 4.79 mm to (43.1, 76.3)
- moved C1 1.54 mm to (135.8, 100.1)
- turned SW1 to 0 degrees
Routing:
- net GND: track 0.00 -> 225.7 mm, vias 0 -> 6
- net Net-(R3-Pad1): track 0.00 -> 127.3 mm, vias 0 -> 4
- net D+: track 0.00 -> 18.2 mm, vias 0 -> 2
- net VCC: track 0.00 -> 12.6 mm, vias 0 -> 2
- net D-: track 0.00 -> 12.1 mm, vias 0 -> 2
- net +5V: track 0.00 -> 9.60 mm
- net row0: track 224.9 -> 230.0 mm
- net Net-(D1-Pad2): track 7.93 -> 7.30 mm

Commit message: Finished routing
Parts:
- moved C1 0.51 mm to (135.3, 100.1)
- moved C4 0.13 mm to (140.1, 107.4)
Connections:
- U1 pad 11: Net-(U1-Pad11) -> col5
- U1 pad 12: Net-(U1-Pad12) -> row0
- U1 pad 21: Net-(U1-Pad21) -> row1
- U1 pad 22: Net-(U1-Pad22) -> col6
- U1 pad 25: Net-(U1-Pad25) -> col11
- U1 pad 26: Net-(U1-Pad26) -> col10
- U1 pad 27: Net-(U1-Pad27) -> col9
- U1 pad 28: Net-(U1-Pad28) -> col8
- U1 pad 29: Net-(U1-Pad29) -> col7
- U1 pad 31: Net-(U1-Pad31) -> row3
- U1 pad 32: Net-(U1-Pad32) -> row2
- U1 pad 37: Net-(U1-Pad37) -> col4
- U1 pad 38: Net-(U1-Pad38) -> col3
- U1 pad 39: Net-(U1-Pad39) -> col2
- U1 pad 40: Net-(U1-Pad40) -> col1
- U1 pad 41: Net-(U1-Pad41) -> col0
Routing:
- net +5V: track 9.60 -> 222.2 mm, vias 0 -> 12
- net col0: track 57.2 -> 178.7 mm, vias 0 -> 10
- net Net-(R1-Pad1): track 0.00 -> 114.4 mm, vias 0 -> 4
- net Net-(R2-Pad1): track 0.00 -> 110.7 mm, vias 0 -> 4
- net col1: track 57.2 -> 156.0 mm, vias 0 -> 8
- net col11: track 57.2 -> 153.3 mm, vias 0 -> 3
- net col2: track 57.2 -> 142.0 mm, vias 0 -> 3
- net GND: track 225.7 -> 307.3 mm
- net col10: track 57.5 -> 134.6 mm, vias 0 -> 3
- net col3: track 57.2 -> 125.5 mm, vias 0 -> 3
- net col9: track 57.2 -> 115.3 mm, vias 0 -> 1
- net row3: track 241.6 -> 285.7 mm, vias 0 -> 2
- net col4: track 58.1 -> 97.5 mm, vias 0 -> 4
- net col8: track 57.3 -> 96.3 mm, vias 0 -> 1
- net row2: track 230.7 -> 254.0 mm
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