File: PCB Design.kicad_pcb (KiCad board)
At the start: 2 copper layers, 228.6 x 76.2 mm, 112 parts, among them SW1 SW_Push, U1 ATmega32U4-AU, Y1 16MHz

Commit message: Figuring out routing and ground fill
Routing:
- added copper zone on B.Cu, net GND
Other:
- board text added: "Diman V1"
Changed lines of the file:
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@@
   (general
     (thickness 1.6)
-    (drawings 8)
+    (drawings 9)
     (tracks 898)
     (zones 0)
@@
     )
   )
+  (gr_text "Diman V1" (at 39.37 136.017) (layer F.SilkS)
+    (effects (font (size 1.27 1.27) (thickness 0.1778)))
+  )
   (gr_line (start 32.16275 62.865) (end 256.00025 62.865) (layer Edge.Cuts) (width 0.05))
   (gr_line (start 29.7815 136.68375) (end 29.7815 65.24625) (layer Edge.Cuts) (width 0.05))
@@
   (segment (start 245.0465 88.9) (end 245.0465 96.3295) (width 0.254) (layer F.Cu) (net 87))
   (segment (start 245.0465 96.3295) (end 245.0465 105.18) (width 0.254) (layer F.Cu) (net 87))
+  (zone (net 1) (net_name GND) (layer B.Cu) (hatch edge 0.508)
+    (connect_pads (clearance 0.508))
+    (min_thickness 0.254)
+    (fill yes (arc_segments 32) (thermal_gap 0.508) (thermal_bridge_width 0.508))
+    (polygon
+      (pts
+        (xy 149.352 78.994) (xy 137.668 78.867) (xy 138.303 84.455) (xy 149.352 84.709)
+      )
+    )
+  )
 )
